Commit message: working differential drive

File: weeding_robot_description/urdf/weeding_robot.xacro (robot description, xacro)
@@ -1,4 +1,5 @@
 <?xml version="1.0"?>
-<robot name="weeding_robot">
+<robot name="weeding_robot" xmlns:xacro="http://www.ros.org/wiki/xacro">
+<xacro:include filename="$(find weeding_robot_description)/urdf/weeding_robot.gazebo.xacro" />
     <material name="grey">
         <color rgba="0.75 0.75 0.75 1"/>
@@ -13,12 +14,4 @@
         <color rgba="0 0.8 0 1"/>
     </material>
-    <!--gazebo plugin for simulation-->
-    <gazebo>
-        <plugin name="gazebo_ros_control" filename="libgazebo_ros_control.so">
-            <robotNamespace>/weeding_robot</robotNamespace>
-            <robotSimType>gazebo_ros_control/DefaultRobotHWSim</robotSimType>
-            <legacyModeNS>true</legacyModeNS>
-        </plugin>
-    </gazebo>
 	<!-- * * * Link Definitions * * * -->
     <link name="base_footprint"/>
@@ -71,5 +64,5 @@
     	<parent link="base_link"/>
     	<child link="left_wheel"/>
-        <origin xyz="-0.572 0.195 -0.03" rpy="0 0 0"/>
+        <origin xyz="-0.572 0.195 -0.03" rpy="0 3.14 0"/>
         <axis xyz="1 0 0"/>
 	</joint>
@@ -107,5 +100,5 @@
     	<parent link="base_link"/>
     	<child link="right_wheel"/>
-        <origin xyz="0.572 0.195 -0.03" rpy="0 0 0"/>
+        <origin xyz="0.572 0.195 -0.03" rpy="0 3.14 0"/>
         <axis xyz="1 0 0"/>
 	</joint>
@@ -146,32 +139,3 @@
         <axis xyz="1 0 0"/>
 	</joint>
-    <gazebo reference="left_wheel">
-        <mu1>0.1</mu1>
-        <mu2>0.1</mu2>
-        <kp>500000.0</kp>
-        <kd>10.0</kd>
-        <minDepth>0.001</minDepth>
-        <maxVel>0.1</maxVel>
-        <fdir1>1 0 0</fdir1>
-        <material>Gazebo/FlatBlack</material>
-     </gazebo>
-    <gazebo reference="right_wheel">
-        <mu1>0.1</mu1>
-        <mu2>0.1</mu2>
-        <kp>500000.0</kp>
-        <kd>10.0</kd>
-        <minDepth>0.001</minDepth>
-        <maxVel>0.1</maxVel>
-        <fdir1>1 0 0</fdir1>
-        <material>Gazebo/FlatBlack</material>
-    </gazebo>
-    <gazebo reference="back_wheel">
-        <mu1>0.1</mu1>
-        <mu2>0.1</mu2>
-        <kp>1000000.0</kp>
-        <kd>100.0</kd>
-        <minDepth>0.001</minDepth>
-        <maxVel>1.0</maxVel>
-        <material>Gazebo/FlatBlack</material>
-    </gazebo>
 </robot>

Commit message: new odom tf using ekf localization node.

File: weeding_robot_description/urdf/weeding_robot.xacro (robot description, xacro)
@@ -19,5 +19,5 @@
         <parent link="base_footprint"/>
         <child link="base_link"/>
-        <origin xyz="0.0 0.0 0.150" rpy="0 0 -1.57"/>
+        <origin xyz="0.0 0.0 0.150" rpy="0 0 0"/>
     </joint>
     <link name="base_link">
@@ -28,5 +28,5 @@
         </inertial>
         <collision>
-            <origin rpy="1.57 0 0" xyz="-0.5 0.345 0"/>
+            <origin rpy="1.57 0 -1.57" xyz="0.345 0.5 0"/>
             <geometry>
                 <mesh filename="package://weeding_robot_description/models/BodycollisionBox.STL" scale="0.001 0.001 0.001"/>
@@ -34,5 +34,5 @@
         </collision>
         <visual>
-            <origin rpy="1.57 0 0" xyz="-0.585 0.345 -0.082"/>
+            <origin rpy="1.57 0 -1.57" xyz="0.345 0.585  -0.082"/>
             <geometry>
                 <mesh filename="package://weeding_robot_description/models/WeedingRobotBodyV3.STL" scale="0.001 0.001 0.001"/>
@@ -64,5 +64,5 @@
     	<parent link="base_link"/>
     	<child link="left_wheel"/>
-        <origin xyz="-0.572 0.195 -0.03" rpy="0 3.14 0"/>
+        <origin xyz="0.195 0.572 -0.03" rpy="0 3.14 -1.57"/>
         <axis xyz="1 0 0"/>
 	</joint>
@@ -100,5 +100,5 @@
     	<parent link="base_link"/>
     	<child link="right_wheel"/>
-        <origin xyz="0.572 0.195 -0.03" rpy="0 3.14 0"/>
+        <origin xyz="0.195 -0.572 -0.03" rpy="0 3.14 -1.57"/>
         <axis xyz="1 0 0"/>
 	</joint>
@@ -136,5 +136,5 @@
     	<parent link="base_link"/>
     	<child link="back_wheel"/>
-        <origin xyz="0 -0.63 -0.085" rpy="0 0 0"/>
+        <origin xyz="-0.63 0 -0.085" rpy="0 0 -1.57"/>
         <axis xyz="1 0 0"/>
 	</joint>
