Commit message: remove unused stuff and update robot urdf

File: weeding_robot_description/urdf/weeding_robot.gazebo.xacro (robot description, xacro)
@@ -35,6 +35,6 @@
     </gazebo>
     <gazebo reference="left_wheel">
-        <mu1>0.1</mu1>
-        <mu2>0.1</mu2>
+        <mu1>1</mu1>
+        <mu2>1</mu2>
         <kp>500000.0</kp>
         <kd>10.0</kd>
@@ -45,6 +45,6 @@
      </gazebo>
     <gazebo reference="right_wheel">
-        <mu1>0.1</mu1>
-        <mu2>0.1</mu2>
+        <mu1>1</mu1>
+        <mu2>1</mu2>
         <kp>500000.0</kp>
         <kd>10.0</kd>
@@ -55,6 +55,6 @@
     </gazebo>
     <gazebo reference="back_wheel">
-        <mu1>0.1</mu1>
-        <mu2>0.1</mu2>
+        <mu1>0.01</mu1>
+        <mu2>0.01</mu2>
         <kp>1000000.0</kp>
         <kd>100.0</kd>

File: weeding_robot_description/urdf/weeding_robot.xacro (robot description, xacro)
@@ -24,6 +24,6 @@
         <inertial>
             <origin xyz="0 0 0" rpy="0 0 0"/>
-            <mass value="5" />
-            <inertia ixx="0.417041666667" ixy="0.0" ixz="0.0" iyy="0.833333333333" iyz="0.0" izz="0.417041666667"/>
+            <mass value="30" />
+            <inertia ixx="3.4" ixy="0.0" ixz="0.0" iyy="3.4" iyz="0.0" izz="5.0"/>
         </inertial>
         <collision>

Commit message: setup

File: weeding_robot_description/urdf/weeding_robot.gazebo.xacro (robot description, xacro)
@@ -2,58 +2,23 @@
 <robot xmlns:xacro="http://www.ros.org/wiki/xacro" name="weeding_robot" >
     <gazebo>
-        <plugin name="gazebo_ros_control" filename="libgazebo_ros_control.so">
-            <legacyModeNS>true</legacyModeNS>
-            <robotNamespace>/weeding_robot</robotNamespace>
-        </plugin>
-        <!--plugin name="differential_drive_controller" filename="libgazebo_ros_diff_drive.so">
-            <legacyMode>true</legacyMode>
+        <plugin name="differential_drive_controller" filename="libgazebo_ros_diff_drive.so">
+            <legacyMode>false</legacyMode>
             <alwaysOn>true</alwaysOn>
             <publishWheelTF>true</publishWheelTF>
-            <publishTf>true</publishTf>
-            <wheelSeparation>1.1</wheelSeparation>
-            <wheelDiameter>0.34</wheelDiameter>
+            <publishTf>1</publishTf>
             <publishWheelJointState>true</publishWheelJointState>
             <updateRate>100.0</updateRate>
             <leftJoint>left_wheel_joint</leftJoint>
             <rightJoint>right_wheel_joint</rightJoint>
+            <wheelSeparation>1.1</wheelSeparation>
+            <wheelDiameter>0.34</wheelDiameter>
             <wheelAcceleration>1.0</wheelAcceleration>
-            <wheelTorque> 5.0 </wheelTorque>
             <torque>20</torque>
             <commandTopic>/weeding_robot/cmd_vel</commandTopic>
-            <odometrySource>world</odometrySource>
-            <odometryTopic>/odom</odometryTopic>
-            <odometryFrame>/odom</odometryFrame>
-            <robotBaseFrame>/base_footprint</robotBaseFrame>
-            <publishOdomTF> true </publishOdomTF>
-            <rosDebugLevel> na </rosDebugLevel>
-        </plugin-->
+            <odometryTopic>odom</odometryTopic>
+            <odometryFrame>odom</odometryFrame>
+            <robotBaseFrame>base_link</robotBaseFrame>
+        </plugin>
     </gazebo>
-    <!-- differential drive setting from turtlebot:
-       <gazebo>
-      <plugin filename="libgazebo_ros_diff_drive.so" name="differential_drive_controller">
-         <alwaysOn>true</alwaysOn>
-         <updateRate>20</updateRate>
-         <publishTf> true </publishTf>
-         <leftJoint>wheel_right_joint</leftJoint>
-         <rightJoint>wheel_left_joint</rightJoint>
-         <wheelSeparation>.230</wheelSeparation>
-         <wheelDiameter>0.070</wheelDiameter>
-         <torque>5.0</torque>
-         <commandTopic>/cmd_vel</commandTopic>
-         <odometrySource>world</odometrySource> # 'encoder' instead of 'world' is also possible
-         <odometryTopic>/odom</odometryTopic> # relative/name ,  /global/name
-         <odometryFrame>/odom</odometryFrame>
-         <robotBaseFrame>/base_footprint</robotBaseFrame>
-         <publishOdomTF> true </publishOdomTF>
-         <publishWheelJointState>true</publishWheelJointState>
-        # Set to true to publish transforms for the wheel links, defaults to false
-         <publishWheelTF>true</publishWheelTF>
-         <wheelAcceleration> 0 </wheelAcceleration>
-         <wheelTorque> 5.0 </wheelTorque>
-         <legacyMode>true</legacyMode>
-         <rosDebugLevel> na </rosDebugLevel> #<rosDebugLevel>Debug</rosDebugLevel>
-      </plugin>
-   </gazebo>
-    -->
     <gazebo>
         <plugin name="gazebo_ros_imu_controller" filename="libgazebo_ros_imu.so">

File: weeding_robot_description/urdf/weeding_robot.xacro (robot description, xacro)
@@ -67,14 +67,4 @@
         <axis xyz="1 0 0"/>
 	</joint>
-    <transmission name="left_wheel_tran">
-        <type>transmission_interface/SimpleTransmission</type>
-        <joint name="left_wheel_joint">
-            <hardwareInterface>hardware_interface/VelocityJointInterface</hardwareInterface>
-        </joint>
-        <actuator name="left_motor">
-            <hardwareInterface>hardware_interface/VelocityJointInterface</hardwareInterface>
-            <mechanicalReduction>1</mechanicalReduction>
-        </actuator>
-    </transmission>
     <link name="right_wheel">
         <inertial>
@@ -103,14 +93,4 @@
         <axis xyz="1 0 0"/>
 	</joint>
-    <transmission name="right_wheel_tran">
-        <type>transmission_interface/SimpleTransmission</type>
-        <joint name="right_wheel_joint">
-            <hardwareInterface>hardware_interface/VelocityJointInterface</hardwareInterface>
-        </joint>
-        <actuator name="right_motor">
-            <hardwareInterface>hardware_interface/VelocityJointInterface</hardwareInterface>
-            <mechanicalReduction>1</mechanicalReduction>
-        </actuator>
-    </transmission>
     <link name="back_wheel">
         <inertial>

Commit message: setup

File: weeding_robot_description/urdf/weeding_robot.gazebo.xacro (robot description, xacro)
@@ -1,9 +1,15 @@
 <?xml version="1.0"?>
 <robot xmlns:xacro="http://www.ros.org/wiki/xacro" name="weeding_robot" >
+    <gazebo>
+        <plugin name="gazebo_ros_control" filename="libgazebo_ros_control.so">
+            <legacyModeNS>false</legacyModeNS>
+            <robotNamespace>/weeding_robot</robotNamespace>
+        </plugin>
+    </gazebo>
     <gazebo>
         <plugin name="differential_drive_controller" filename="libgazebo_ros_diff_drive.so">
             <legacyMode>false</legacyMode>
             <alwaysOn>true</alwaysOn>
-            <publishWheelTF>true</publishWheelTF>
+            <publishWheelTF>false</publishWheelTF>
             <publishTf>1</publishTf>
             <publishWheelJointState>true</publishWheelJointState>
@@ -18,5 +24,5 @@
             <odometryTopic>odom</odometryTopic>
             <odometryFrame>odom</odometryFrame>
-            <robotBaseFrame>base_link</robotBaseFrame>
+            <robotBaseFrame>base_footprint</robotBaseFrame>
         </plugin>
     </gazebo>

File: weeding_robot_description/urdf/weeding_robot.xacro (robot description, xacro)
@@ -67,4 +67,14 @@
         <axis xyz="1 0 0"/>
 	</joint>
+    <transmission name="left_wheel_tran">
+        <type>transmission_interface/SimpleTransmission</type>
+        <joint name="left_wheel_joint">
+            <hardwareInterface>hardware_interface/VelocityJointInterface</hardwareInterface>
+        </joint>
+        <actuator name="left_motor">
+            <hardwareInterface>hardware_interface/VelocityJointInterface</hardwareInterface>
+            <mechanicalReduction>1</mechanicalReduction>
+        </actuator>
+    </transmission>
     <link name="right_wheel">
         <inertial>
@@ -93,4 +103,14 @@
         <axis xyz="1 0 0"/>
 	</joint>
+    <transmission name="right_wheel_tran">
+        <type>transmission_interface/SimpleTransmission</type>
+        <joint name="right_wheel_joint">
+            <hardwareInterface>hardware_interface/VelocityJointInterface</hardwareInterface>
+        </joint>
+        <actuator name="right_motor">
+            <hardwareInterface>hardware_interface/VelocityJointInterface</hardwareInterface>
+            <mechanicalReduction>1</mechanicalReduction>
+        </actuator>
+    </transmission>
     <link name="back_wheel">
         <inertial>

Commit message: fix footprint

File: weeding_robot_description/urdf/weeding_robot.gazebo.xacro (robot description, xacro)
@@ -29,5 +29,5 @@
             <topicName>gps/fix</topicName>
             <velocityTopicName>gps/fix_velocity</velocityTopicName>
-            <drift>5.0 5.0 5.0</drift>
+            <drift>0 0 0</drift>
             <gaussianNoise>0.1 0.1 0.1</gaussianNoise>
             <velocityDrift>0 0 0</velocityDrift>

File: weeding_robot_description/urdf/weeding_robot.xacro (robot description, xacro)
@@ -19,5 +19,5 @@
         <parent link="base_footprint"/>
         <child link="base_link"/>
-        <origin xyz="0.0 0.0 0.010" rpy="0 0 0"/>
+        <origin xyz="0.0 0.0 0.150" rpy="0 0 -1.57"/>
     </joint>
     <link name="base_link">

Commit message: change tilt angel

File: weeding_robot_description/urdf/weeding_robot.gazebo.xacro (robot description, xacro)
@@ -12,5 +12,6 @@
             <topicName>imu/data</topicName>
             <serviceName>imu/service</serviceName>
-            <bodyName>base_link</bodyName>
+            <bodyName>base_imu_link</bodyName>
+            <frameName>base_imu_link</frameName>
             <gaussianNoise>0</gaussianNoise>
             <rpyOffsets>0 0 0</rpyOffsets>

File: weeding_robot_description/urdf/weeding_robot.xacro (robot description, xacro)
@@ -139,3 +139,27 @@
         <axis xyz="1 0 0"/>
 	</joint>
+    <link name="base_imu_link">
+    <inertial>
+        <mass value="0.001"/>
+        <origin rpy="0 0 0" xyz="0 0 0"/>
+        <inertia ixx="0.0001" ixy="0" ixz="0" iyy="0.000001" iyz="0" izz="0.0001"/>
+    </inertial>
+    <visual>
+        <origin rpy="0 0 0" xyz="0 0 0"/>
+        <geometry>
+        <box size="0.001 0.001 0.001"/>
+        </geometry>
+    </visual>
+    <collision>
+        <origin rpy="0 0 0" xyz="0 0 0"/>
+        <geometry>
+        <box size=".001 .001 .001"/>
+        </geometry>
+    </collision>
+    </link>
+    <joint name="base_imu_joint" type="fixed">
+        <parent link="base_link"/>
+        <child link="base_imu_link"/>
+        <origin xyz="0.3 0.0 0" rpy="3.14 0 1.57"/>
+    </joint>
 </robot>

File: weeding_robot_description/urdf/weeding_robot_simple.xacro (robot description, xacro)
@@ -18,5 +18,5 @@
         <parent link="base_footprint"/>
         <child link="base_link"/>
-        <origin xyz="0.0 0.0 0.150" rpy="0 0 0"/>
+        <origin xyz="0.0 0.0 0.150" rpy="0 0.13962634 0"/>
     </joint>
     <link name="base_link">
