Commit message: add a simplified urdf to solve the wheed detach issue. not ideal solution

File: weeding_robot_description/urdf/weeding_robot_simple.xacro (robot description, xacro)
@@ -1,5 +1,4 @@
 <?xml version="1.0"?>
 <robot name="weeding_robot" xmlns:xacro="http://www.ros.org/wiki/xacro">
-<xacro:include filename="$(find weeding_robot_description)/urdf/weeding_robot.gazebo.xacro" />
     <material name="grey">
         <color rgba="0.75 0.75 0.75 1"/>
@@ -61,5 +60,5 @@
         </visual>
     </link>
-    <joint name="left_wheel_joint" type="continuous">
+    <joint name="left_wheel_joint" type="fixed">
     	<parent link="base_link"/>
     	<child link="left_wheel"/>
@@ -67,14 +66,4 @@
         <axis xyz="1 0 0"/>
 	</joint>
-    <transmission name="left_wheel_tran">
-        <type>transmission_interface/SimpleTransmission</type>
-        <joint name="left_wheel_joint">
-            <hardwareInterface>hardware_interface/VelocityJointInterface</hardwareInterface>
-        </joint>
-        <actuator name="left_motor">
-            <hardwareInterface>hardware_interface/VelocityJointInterface</hardwareInterface>
-            <mechanicalReduction>1</mechanicalReduction>
-        </actuator>
-    </transmission>
     <link name="right_wheel">
         <inertial>
@@ -97,5 +86,5 @@
         </visual>
     </link>
-    <joint name="right_wheel_joint" type="continuous">
+    <joint name="right_wheel_joint" type="fixed">
     	<parent link="base_link"/>
     	<child link="right_wheel"/>
@@ -103,14 +92,4 @@
         <axis xyz="1 0 0"/>
 	</joint>
-    <transmission name="right_wheel_tran">
-        <type>transmission_interface/SimpleTransmission</type>
-        <joint name="right_wheel_joint">
-            <hardwareInterface>hardware_interface/VelocityJointInterface</hardwareInterface>
-        </joint>
-        <actuator name="right_motor">
-            <hardwareInterface>hardware_interface/VelocityJointInterface</hardwareInterface>
-            <mechanicalReduction>1</mechanicalReduction>
-        </actuator>
-    </transmission>
     <link name="back_wheel">
         <inertial>

Commit message: add imu base link

File: weeding_robot_description/urdf/weeding_robot_simple.xacro (robot description, xacro)
@@ -118,3 +118,10 @@
         <axis xyz="1 0 0"/>
 	</joint>
+    <link name="base_imu_link">
+    </link>
+    <joint name="base_imu_joint" type="fixed">
+        <parent link="base_link"/>
+        <child link="base_imu_link"/>
+        <origin xyz="0.3 0.0 0" rpy="0 0 0"/>
+    </joint>
 </robot>

Commit message: change imu orientation

File: weeding_robot_description/urdf/weeding_robot_simple.xacro (robot description, xacro)
@@ -123,5 +123,5 @@
         <parent link="base_link"/>
         <child link="base_imu_link"/>
-        <origin xyz="0.3 0.0 0" rpy="0 0 0"/>
+        <origin xyz="0.3 0.0 0" rpy="3.14 0 1.57"/>
     </joint>
 </robot>

Commit message: change base imu link

File: weeding_robot_description/urdf/weeding_robot_simple.xacro (robot description, xacro)
@@ -123,5 +123,5 @@
         <parent link="base_link"/>
         <child link="base_imu_link"/>
-        <origin xyz="0.3 0.0 0" rpy="3.14 0 1.57"/>
+        <origin xyz="0.3 0.0 0" rpy="0 0 0"/>
     </joint>
 </robot>
